Commit message: add a cylinder tool for the project

File: robot/universal_robot/fmauch_universal_robot/ur_gazebo/urdf/ur.xacro (robot description, xacro)
@@ -67,3 +67,27 @@
     <origin xyz="0 0 0" rpy="0 0 0"/>
   </joint>
+  <link name="tool_cylinder0_link">
+    <visual>
+      <geometry>
+        <cylinder length="0.05" radius="0.005"/>
+      </geometry>
+    </visual>
+  </link>
+  <joint name="tool_joint0" type="fixed">
+    <parent link="tool0"/>
+    <child link="tool_cylinder0_link"/>
+    <origin xyz="0 0 0.025" rpy="0 0 0"/>
+  </joint>
+  <link name="tool_cylinder1_link">
+    <visual>
+      <geometry>
+        <cylinder length="0.001" radius="0.01"/>
+      </geometry>
+    </visual>
+  </link>
+  <joint name="tool_joint1" type="fixed">
+    <parent link="tool_cylinder0_link"/>
+    <child link="tool_cylinder1_link"/>
+    <origin xyz="0 0 0.025" rpy="0 0 0"/>
+  </joint>
 </robot>

Commit message: add two depth camera to detect the desired work range

File: robot/universal_robot/fmauch_universal_robot/ur_gazebo/urdf/ur.xacro (robot description, xacro)
@@ -91,3 +91,135 @@
     <origin xyz="0 0 0.025" rpy="0 0 0"/>
   </joint>
+  <joint name="camera_joint1" type="fixed">
+    <axis xyz="0 1 0" />
+    <origin xyz="0.7 0 0.5" rpy="0.0 1.5707963 0.0"/>
+    <parent link="world"/>
+    <child link="camera_link1"/>
+  </joint>
+  <link name="camera_link1">
+    <collision>
+      <origin xyz="0 0 0" rpy="0 0 0"/>
+      <geometry>
+        <box size="0.0 0.0 0.0"/>
+      </geometry>
+    </collision>
+    <visual>
+      <origin xyz="0 0 0" rpy="0 0 0"/>
+      <geometry>
+        <box size="0.025 0.025 0.025"/>
+      </geometry>
+    </visual>
+    <inertial>
+      <mass value="1e-5" />
+      <origin xyz="0 0 0" rpy="0 0 0"/>
+      <inertia ixx="1e-6" ixy="0" ixz="0" iyy="1e-6" iyz="0" izz="1e-6" />
+    </inertial>
+  </link>
+  <gazebo reference="camera_link1">
+    <sensor name="camera1" type="depth">
+      <update_rate>20</update_rate>
+      <camera>
+        <horizontal_fov>1.047198</horizontal_fov>
+        <image>
+          <width>640</width>
+          <height>480</height>
+          <format>R8G8B8</format>
+        </image>
+        <clip>
+          <near>0.05</near>
+          <far>3</far>
+        </clip>
+      </camera>
+      <plugin name="camera1_controller" filename="libgazebo_ros_openni_kinect.so">
+        <baseline>0.2</baseline>
+        <alwaysOn>true</alwaysOn>
+        <updateRate>1.0</updateRate>
+        <cameraName>camera1_ir</cameraName>
+        <imageTopicName>/camera1/color/image_raw</imageTopicName>
+        <cameraInfoTopicName>/camera1/color/camera_info</cameraInfoTopicName>
+        <depthImageTopicName>/camera1/depth/image_raw</depthImageTopicName>
+        <depthImageInfoTopicName>/camera1/depth/camera_info</depthImageInfoTopicName>
+        <pointCloudTopicName>/camera1/depth/points</pointCloudTopicName>
+        <frameName>camera_link1</frameName>
+        <pointCloudCutoff>0.5</pointCloudCutoff>
+        <pointCloudCutoffMax>3.0</pointCloudCutoffMax>
+        <distortionK1>0.00000001</distortionK1>
+        <distortionK2>0.00000001</distortionK2>
+        <distortionK3>0.00000001</distortionK3>
+        <distortionT1>0.00000001</distortionT1>
+        <distortionT2>0.00000001</distortionT2>
+        <CxPrime>0</CxPrime>
+        <Cx>0</Cx>
+        <Cy>0</Cy>
+        <focalLength>0</focalLength>
+        <hackBaseline>0</hackBaseline>
+      </plugin>
+    </sensor>
+  </gazebo>
+  <joint name="camera_joint2" type="fixed">
+    <axis xyz="0 1 0" />
+    <origin xyz="-0.7 0 0.5" rpy="0.0 1.5707963 0.0"/>
+    <parent link="world"/>
+    <child link="camera_link2"/>
+  </joint>
+  <link name="camera_link2">
+    <collision>
+      <origin xyz="0 0 0" rpy="0 0 0"/>
+      <geometry>
+        <box size="0.0 0.0 0.0"/>
+      </geometry>
+    </collision>
+    <visual>
+      <origin xyz="0 0 0" rpy="0 0 0"/>
+      <geometry>
+        <box size="0.025 0.025 0.025"/>
+      </geometry>
+    </visual>
+    <inertial>
+      <mass value="1e-5" />
+      <origin xyz="0 0 0" rpy="0 0 0"/>
+      <inertia ixx="1e-6" ixy="0" ixz="0" iyy="1e-6" iyz="0" izz="1e-6" />
+    </inertial>
+  </link>
+  <gazebo reference="camera_link2">
+    <sensor name="camera2" type="depth">
+      <update_rate>20</update_rate>
+      <camera>
+        <horizontal_fov>1.047198</horizontal_fov>
+        <image>
+          <width>640</width>
+          <height>480</height>
+          <format>R8G8B8</format>
+        </image>
+        <clip>
+          <near>0.05</near>
+          <far>3</far>
+        </clip>
+      </camera>
+      <plugin name="camera2_controller" filename="libgazebo_ros_openni_kinect.so">
+        <baseline>0.2</baseline>
+        <alwaysOn>true</alwaysOn>
+        <updateRate>1.0</updateRate>
+        <cameraName>camera2_ir</cameraName>
+        <imageTopicName>/camera2/color/image_raw</imageTopicName>
+        <cameraInfoTopicName>/camera2/color/camera_info</cameraInfoTopicName>
+        <depthImageTopicName>/camera2/depth/image_raw</depthImageTopicName>
+        <depthImageInfoTopicName>/camera2/depth/camera_info</depthImageInfoTopicName>
+        <pointCloudTopicName>/camera2/depth/points</pointCloudTopicName>
+        <frameName>camera_link2</frameName>
+        <pointCloudCutoff>0.5</pointCloudCutoff>
+        <pointCloudCutoffMax>3.0</pointCloudCutoffMax>
+        <distortionK1>0.00000001</distortionK1>
+        <distortionK2>0.00000001</distortionK2>
+        <distortionK3>0.00000001</distortionK3>
+        <distortionT1>0.00000001</distortionT1>
+        <distortionT2>0.00000001</distortionT2>
+        <CxPrime>0</CxPrime>
+        <Cx>0</Cx>
+        <Cy>0</Cy>
+        <focalLength>0</focalLength>
+        <hackBaseline>0</hackBaseline>
+      </plugin>
+    </sensor>
+  </gazebo>
 </robot>
